File: breadboard_power_supply.kicad_sch (KiCad schematic)
At the start: 19 parts, among them J1 PJ-059AH, J11 Conn_01x12_Male, J13 Conn_01x04_Male, J4 Screw_Terminal_01x06, J6 Conn_01x03_Male, J7 Screw_Terminal_01x02, U1 LM7805_TO220, U2 LM317_TO-220

Commit message: BOM
Parts:
- J11: value Conn_01x12_Male -> Conn_01x12
- J13: value Conn_01x04_Male -> Conn_01x04; PURPOSE FAN_CONTRO_PINHEADS -> FAN_CONTRO_PINSOCKETS
Changed lines of the file:
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@@
     (in_bom yes) (on_board yes)
     (property "Reference" "J13" (id 0) (at 191.135 139.7 0))
-    (property "Value" "Conn_01x04_Male" (id 1) (at 191.135 142.24 0))
+    (property "Value" "Conn_01x04" (id 1) (at 191.135 142.24 0))
     (property "Footprint" "Connector_PinSocket_2.54mm:PinSocket_1x04_P2.54mm_Vertical" (id 2) (at 190.5 147.32 0)
       (effects (font (size 1.27 1.27)) hide)
@@
       (effects (font (size 1.27 1.27)) hide)
     )
-    (property "PURPOSE" "FAN_CONTRO_PINHEADS" (id 4) (at 190.5 157.48 0))
+    (property "PURPOSE" "FAN_CONTRO_PINSOCKETS" (id 4) (at 190.5 157.48 0))
     (pin "1")
     (pin "2")
@@
     (in_bom yes) (on_board yes)
     (property "Reference" "J11" (id 0) (at 69.215 139.7 0))
-    (property "Value" "Conn_01x12_Male" (id 1) (at 69.215 142.24 0))
+    (property "Value" "Conn_01x12" (id 1) (at 69.215 142.24 0))
     (property "Footprint" "Connector_PinSocket_2.54mm:PinSocket_1x12_P2.54mm_Vertical" (id 2) (at 68.58 157.48 0)
       (effects (font (size 1.27 1.27)) hide)
@@
     )
     (path "/e37b0ec1-e6e0-41cc-abe1-ad47cc32e2d2"
-      (reference "J11") (unit 1) (value "Conn_01x12_Male") (footprint "Connector_PinSocket_2.54mm:PinSocket_1x12_P2.54mm_Vertical")
+      (reference "J11") (unit 1) (value "Conn_01x12") (footprint "Connector_PinSocket_2.54mm:PinSocket_1x12_P2.54mm_Vertical")
     )
     (path "/3c44e781-1190-4e9e-8bbc-c825cbc80c09/e48c6b79-23e7-490e-8d34-0153e7625f18"
@@
     )
     (path "/7ca95307-4877-4e7a-bcd4-ef48e48df98e"
-      (reference "J13") (unit 1) (value "Conn_01x04_Male") (footprint "Connector_PinSocket_2.54mm:PinSocket_1x04_P2.54mm_Vertical")
+      (reference "J13") (unit 1) (value "Conn_01x04") (footprint "Connector_PinSocket_2.54mm:PinSocket_1x04_P2.54mm_Vertical")
     )
     (path "/3c44e781-1190-4e9e-8bbc-c825cbc80c09/2a385001-5407-4245-8e25-035c6053c743"

Commit message: BOM
Parts:
- R2: value 330 -> 470
Changed lines of the file:
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@@
       (effects (font (size 1.27 1.27) italic) hide)
     )
-    (property "Datasheet" "https://www.onsemi.cn/PowerSolutions/document/MC7800-D.PDF" (id 3) (at 124.46 46.99 0)
+    (property "Datasheet" "https://www.tme.eu/Document/8aa8ed83dc2f8e8a5f3ad4a71fd201bc/lm7805.pdf" (id 3) (at 124.46 46.99 0)
       (effects (font (size 1.27 1.27)) hide)
     )
@@
       (effects (font (size 1.27 1.27)) (justify right))
     )
-    (property "Value" "330" (id 1) (at 73.66 104.1399 0)
+    (property "Value" "470" (id 1) (at 73.66 104.1399 0)
       (effects (font (size 1.27 1.27)) (justify right))
     )
@@
     )
     (path "/6fe50946-2be9-4286-9b3d-a1ad70deb934"
-      (reference "R2") (unit 1) (value "330") (footprint "Resistor_SMD:R_0805_2012Metric")
+      (reference "R2") (unit 1) (value "470") (footprint "Resistor_SMD:R_0805_2012Metric")
     )
     (path "/e6b45546-c8d6-458a-90b9-8ea17a804c93"
